File: pushButton_debounced.brd (EAGLE design)
At the start: 68.6 x 53.3 mm, 3 parts

Commit message: Part One Completed
Parts:
- removed R1: 10k‎Ω, AUTODESK_CIRCUITS_BREADBOARD:0207/10
- removed S1: (no value), AUTODESK_CIRCUITS_BREADBOARD:TL1105
- added D1: (no value), AUTODESK_CIRCUITS_BREADBOARD:LED5MM
- added R3, R4: 1k‎Ω, AUTODESK_CIRCUITS_BREADBOARD:0207/10
- added S3: (no value), AUTODESK_CIRCUITS_BREADBOARD:TL1105
- renumbered U1 to U3
Connections:
- new net N$6: S3.2
- new net N$7: R3.2, S3.3
- new net N$8: R3.1, U3.GND..
- net N$1: now also S3.4, U3.5V; no longer R1.2, S1.3
- net N$2: now also S3.1, U3.2; no longer R1.1, U3.GND..
- net N$3: now also R4.1, U3.13; no longer S1.4, U3.5V
- net N$4: now also D1.A, R4.2; no longer S1.1, U3.2
- net N$5: now also D1.K, U3.GND; no longer S1.2
Changed lines of the file:
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@@
 </autorouter>
 <elements>
-<element value="" name="U1" library="AUTODESK_CIRCUITS_BREADBOARD" package="ARDUINO_UNO" x="5" y="10.08"></element><element value="10k‎Ω" name="R1" library="AUTODESK_CIRCUITS_BREADBOARD" package="0207/10" x="5" y="22.78"></element><element value="" name="S1" library="AUTODESK_CIRCUITS_BREADBOARD" package="TL1105" x="5" y="35.480000000000004"></element></elements>
+<element value="" name="U3" library="AUTODESK_CIRCUITS_BREADBOARD" package="ARDUINO_UNO" x="5" y="10.08"></element><element value="" name="S3" library="AUTODESK_CIRCUITS_BREADBOARD" package="TL1105" x="5" y="22.78"></element><element value="" name="D1" library="AUTODESK_CIRCUITS_BREADBOARD" package="LED5MM" x="5" y="35.480000000000004"></element><element value="1k‎Ω" name="R4" library="AUTODESK_CIRCUITS_BREADBOARD" package="0207/10" x="5" y="48.18"></element><element value="1k‎Ω" name="R3" library="AUTODESK_CIRCUITS_BREADBOARD" package="0207/10" x="5" y="60.879999999999995"></element></elements>
 <signals>
-<signal name="N$1"><contactref element="S1" pad="3"></contactref><contactref element="R1" pad="2"></contactref><wire x1="2.75" y1="32.230000000000004" x2="10.08" y2="22.78" width="0" layer="19" extent="1-1"></wire></signal><signal name="N$2"><contactref element="R1" pad="1"></contactref><contactref element="U1" pad="GND.."></contactref><wire x1="-0.08000000000000007" y1="22.78" x2="45.64" y2="12.620000000000001" width="0" layer="19" extent="1-1"></wire></signal><signal name="N$3"><contactref element="S1" pad="4"></contactref><contactref element="U1" pad="5V"></contactref><wire x1="7.25" y1="32.230000000000004" x2="43.1" y2="12.620000000000001" width="0" layer="19" extent="1-1"></wire></signal><signal name="N$4"><contactref element="U1" pad="2"></contactref><contactref element="S1" pad="1"></contactref><wire x1="63.42" y1="60.879999999999995" x2="2.75" y2="38.730000000000004" width="0" layer="19" extent="1-1"></wire></signal><signal name="N$5"><contactref element="S1" pad="2"></contactref></signal></signals>
+<signal name="N$1"><contactref element="S3" pad="4"></contactref><contactref element="U3" pad="5V"></contactref><wire x1="7.25" y1="19.53" x2="43.1" y2="12.620000000000001" width="0" layer="19" extent="1-1"></wire></signal><signal name="N$2"><contactref element="S3" pad="1"></contactref><contactref element="U3" pad="2"></contactref><wire x1="2.75" y1="26.03" x2="63.42" y2="60.879999999999995" width="0" layer="19" extent="1-1"></wire></signal><signal name="N$3"><contactref element="R4" pad="1"></contactref><contactref element="U3" pad="13"></contactref><wire x1="-0.08000000000000007" y1="48.18" x2="33.956" y2="60.879999999999995" width="0" layer="19" extent="1-1"></wire></signal><signal name="N$4"><contactref element="D1" pad="A"></contactref><contactref element="R4" pad="2"></contactref><wire x1="3.73" y1="35.480000000000004" x2="10.08" y2="48.18" width="0" layer="19" extent="1-1"></wire></signal><signal name="N$5"><contactref element="D1" pad="K"></contactref><contactref element="U3" pad="GND"></contactref><wire x1="6.27" y1="35.480000000000004" x2="31.416" y2="60.879999999999995" width="0" layer="19" extent="1-1"></wire></signal><signal name="N$6"><contactref element="S3" pad="2"></contactref></signal><signal name="N$7"><contactref element="S3" pad="3"></contactref><contactref element="R3" pad="2"></contactref><wire x1="2.75" y1="19.53" x2="10.08" y2="60.879999999999995" width="0" layer="19" extent="1-1"></wire></signal><signal name="N$8"><contactref element="R3" pad="1"></contactref><contactref element="U3" pad="GND.."></contactref><wire x1="-0.08000000000000007" y1="60.879999999999995" x2="45.64" y2="12.620000000000001" width="0" layer="19" extent="1-1"></wire></signal></signals>
 </board>
 </drawing>
