File: servoIR.brd (EAGLE design)
At the start: 68.6 x 53.3 mm, 5 parts

Commit message: task 3(b)
Parts:
- removed D1: (no value), AUTODESK_CIRCUITS_BREADBOARD:LED5MM
- removed R1: 120‎Ω, AUTODESK_CIRCUITS_BREADBOARD:0207/10
Connections:
- removed net N$1 (its old number): R1.1, SERVO1.3, U1.9
- removed net N$5: D1.A, R1.2
- new net N$2: SERVO1.1, U1.GND.., U2.2
- net N$3: now also U1.3, U2.3; no longer D1.K, SERVO1.1, U1.GND.., U2.2
- net N$4: now also SERVO1.3, U1.9; no longer U1.2, U2.3
Changed lines of the file:
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@@
 </autorouter>
 <elements>
-<element value="" name="U1" library="AUTODESK_CIRCUITS_BREADBOARD" package="ARDUINO_UNO" x="5" y="10.08"></element><element value="" name="SERVO1" library="AUTODESK_CIRCUITS_BREADBOARD" package="1X3P-2.54-2.54-11.6-3.0-BLACK-MALE" x="5" y="22.78"></element><element value="" name="U2" library="AUTODESK_CIRCUITS_BREADBOARD" package="1X3P-2.54-2.54-11.6-3.0-BLACK-MALE" x="5" y="35.480000000000004"></element><element value="" name="D1" library="AUTODESK_CIRCUITS_BREADBOARD" package="LED5MM" x="5" y="48.18"></element><element value="120‎Ω" name="R1" library="AUTODESK_CIRCUITS_BREADBOARD" package="0207/10" x="5" y="60.879999999999995"></element></elements>
+<element value="" name="U1" library="AUTODESK_CIRCUITS_BREADBOARD" package="ARDUINO_UNO" x="5" y="10.08"></element><element value="" name="SERVO1" library="AUTODESK_CIRCUITS_BREADBOARD" package="1X3P-2.54-2.54-11.6-3.0-BLACK-MALE" x="5" y="22.78"></element><element value="" name="U2" library="AUTODESK_CIRCUITS_BREADBOARD" package="1X3P-2.54-2.54-11.6-3.0-BLACK-MALE" x="5" y="35.480000000000004"></element></elements>
 <signals>
-<signal name="N$1"><contactref element="SERVO1" pad="3"></contactref><contactref element="U1" pad="9"></contactref><wire x1="5" y1="20.240000000000002" x2="44.116" y2="60.879999999999995" width="0" layer="19" extent="1-1"></wire><contactref element="R1" pad="1"></contactref><wire x1="44.116" y1="60.879999999999995" x2="-0.08000000000000007" y2="60.879999999999995" width="0" layer="19" extent="1-1"></wire></signal><signal name="N$2"><contactref element="SERVO1" pad="2"></contactref><contactref element="U1" pad="5V"></contactref><wire x1="5" y1="22.78" x2="43.1" y2="12.620000000000001" width="0" layer="19" extent="1-1"></wire><contactref element="U2" pad="1"></contactref><wire x1="43.1" y1="12.620000000000001" x2="5" y2="38.02" width="0" layer="19" extent="1-1"></wire></signal><signal name="N$3"><contactref element="U1" pad="GND.."></contactref><contactref element="SERVO1" pad="1"></contactref><wire x1="45.64" y1="12.620000000000001" x2="5" y2="25.32" width="0" layer="19" extent="1-1"></wire><contactref element="U2" pad="2"></contactref><wire x1="5" y1="25.32" x2="5" y2="35.480000000000004" width="0" layer="19" extent="1-1"></wire><contactref element="D1" pad="K"></contactref><wire x1="5" y1="35.480000000000004" x2="6.27" y2="48.18" width="0" layer="19" extent="1-1"></wire></signal><signal name="N$4"><contactref element="U2" pad="3"></contactref><contactref element="U1" pad="2"></contactref><wire x1="5" y1="32.940000000000005" x2="63.42" y2="60.879999999999995" width="0" layer="19" extent="1-1"></wire></signal><signal name="N$5"><contactref element="R1" pad="2"></contactref><contactref element="D1" pad="A"></contactref><wire x1="10.08" y1="60.879999999999995" x2="3.73" y2="48.18" width="0" layer="19" extent="1-1"></wire></signal></signals>
+<signal name="N$1"><contactref element="U1" pad="5V"></contactref><contactref element="U2" pad="1"></contactref><wire x1="43.1" y1="12.620000000000001" x2="5" y2="38.02" width="0" layer="19" extent="1-1"></wire><contactref element="SERVO1" pad="2"></contactref><wire x1="5" y1="38.02" x2="5" y2="22.78" width="0" layer="19" extent="1-1"></wire></signal><signal name="N$2"><contactref element="U1" pad="GND.."></contactref><contactref element="U2" pad="2"></contactref><wire x1="45.64" y1="12.620000000000001" x2="5" y2="35.480000000000004" width="0" layer="19" extent="1-1"></wire><contactref element="SERVO1" pad="1"></contactref><wire x1="5" y1="35.480000000000004" x2="5" y2="25.32" width="0" layer="19" extent="1-1"></wire></signal><signal name="N$3"><contactref element="U2" pad="3"></contactref><contactref element="U1" pad="3"></contactref><wire x1="5" y1="32.940000000000005" x2="60.88" y2="60.879999999999995" width="0" layer="19" extent="1-1"></wire></signal><signal name="N$4"><contactref element="SERVO1" pad="3"></contactref><contactref element="U1" pad="9"></contactref><wire x1="5" y1="20.240000000000002" x2="44.116" y2="60.879999999999995" width="0" layer="19" extent="1-1"></wire></signal></signals>
 </board>
 </drawing>
